Commit message: Added back wheels on Cheesebot

File: catkin_ws/src/myrobot/myrobot_description/urdf/myrobot.xacro (robot description, xacro)
@@ -65,4 +65,12 @@
       <origin xyz="${wheel_base_x} ${-wheel_base_y} ${wheel_base_z}"/>
     </xacro:wheel>
+    <xacro:wheel wheel_prefix="left_back" parent_link="base_link" left_right="-1"
+      radius="${wheel_radius}" width="${wheel_width}" mass="${wheel_mass}">
+      <origin xyz="${-1*wheel_base_x} ${wheel_base_y} ${wheel_base_z}"/>
+    </xacro:wheel>
+    <xacro:wheel wheel_prefix="right_back" parent_link="base_link" left_right="1"
+      radius="${wheel_radius}" width="${wheel_width}" mass="${wheel_mass}">
+      <origin xyz="${-1*wheel_base_x} ${-wheel_base_y} ${wheel_base_z}"/>
+    </xacro:wheel>
     <!--
     <xacro:roller name="front" parent="base_link" radius="${roller_radius}" mass="${roller_mass}">

File: catkin_ws/src/myrobot/myrobot_simulator/urdf/macro.gazebo.xacro (robot description, xacro)
@@ -6,4 +6,12 @@
   </gazebo>
   <gazebo reference="right_wheel">
+    <mu1>4</mu1>
+    <mu2>4</mu2>
+  </gazebo>
+  <gazebo reference="left_back_wheel">
+    <mu1>4</mu1>
+    <mu2>4</mu2>
+  </gazebo>
+  <gazebo reference="right_back_wheel">
     <mu1>4</mu1>
     <mu2>4</mu2>

Commit message: Resized the CheeseBot and fixed LIDAR placement

File: catkin_ws/src/myrobot/myrobot_description/urdf/myrobot.xacro (robot description, xacro)
@@ -2,9 +2,9 @@
 <robot name="myrobot" xmlns:xacro="http://www.ros.org/wiki/xacro">
   <!-- ============ Enter xacro properties here (if you want) =============== -->
-  <xacro:property name="base_size_x" value="0.2"/>
+  <xacro:property name="base_size_x" value="0.17"/>
   <xacro:property name="base_size_y" value="0.15"/>
   <xacro:property name="base_size_z" value="0.07"/>
   <xacro:property name="base_mass" value="2"/>
-  <xacro:property name="wheel_radius" value="0.1"/>
+  <xacro:property name="wheel_radius" value="0.08"/>
   <xacro:property name="wheel_width" value="0.03"/>
   <xacro:property name="wheel_mass" value="0.1"/>
@@ -26,5 +26,5 @@
   <xacro:property name="wheel_base_y" value="${base_size_y/2 + wheel_width/2}"/>
   <!-- <xacro:property name="wheel_base_z" value="${-1 * sqrt((base_size_x*base_size_x) - (wheel_base_x*wheel_base_x))}"/> -->
-  <xacro:property name="wheel_base_z" value="${-0.15198+wheel_radius}"/>
+  <xacro:property name="wheel_base_z" value="${-1 * sqrt((base_size_x*base_size_x) - (wheel_base_x*wheel_base_x))+wheel_radius}"/>
   <xacro:property name="roller_base_x" value="${roller_radius}"/>
   <xacro:property name="roller_base_y" value="0.0"/>
@@ -32,8 +32,8 @@
   <xacro:property name="lidar_base_x" value="0.0"/>
   <xacro:property name="lidar_base_y" value="0.0"/>
-  <xacro:property name="lidar_base_z" value="${base_size_z}"/>
-  <xacro:property name="ir_base_x" value="${base_size_x / 2}"/>
+  <xacro:property name="lidar_base_z" value="${base_size_x + wheel_radius}"/>
+  <xacro:property name="ir_base_x" value="${base_size_x*0.705}"/>
   <xacro:property name="ir_base_y" value="${base_size_y / 2}"/>
-  <xacro:property name="ir_base_z" value="${base_size_z / 2}"/>
+  <xacro:property name="ir_base_z" value="${base_size_x*0.705 + wheel_radius}"/>
   <!-- ============ Including macros and materials =============== -->
   <xacro:include filename="$(find myrobot_description)/urdf/macro.xacro"/>

Commit message: Updated LIDAR python code

File: catkin_ws/src/myrobot/myrobot_description/urdf/myrobot.xacro (robot description, xacro)
@@ -9,6 +9,4 @@
   <xacro:property name="wheel_width" value="0.03"/>
   <xacro:property name="wheel_mass" value="0.1"/>
-  <xacro:property name="roller_radius" value="0.05"/>
-  <xacro:property name="roller_mass" value="0.1"/>
   <xacro:property name="lidar_radius" value="0.002"/>
   <xacro:property name="lidar_width" value="0.002"/>
@@ -27,7 +25,4 @@
   <!-- <xacro:property name="wheel_base_z" value="${-1 * sqrt((base_size_x*base_size_x) - (wheel_base_x*wheel_base_x))}"/> -->
   <xacro:property name="wheel_base_z" value="${-1 * sqrt((base_size_x*base_size_x) - (wheel_base_x*wheel_base_x))+wheel_radius}"/>
-  <xacro:property name="roller_base_x" value="${roller_radius}"/>
-  <xacro:property name="roller_base_y" value="0.0"/>
-  <xacro:property name="roller_base_z" value="0.0"/>
   <xacro:property name="lidar_base_x" value="0.0"/>
   <xacro:property name="lidar_base_y" value="0.0"/>
@@ -48,9 +43,4 @@
   </joint>
     <!-- ============ Enter base_link code here =============== -->
-<!--
-    <link name="base_link">
-      <xacro:make_box sx="${base_size_x}" sy="${base_size_y}" sz="${base_size_z}" mass="${base_mass}" xyz="${base_x} ${base_y} ${base_z}"/>
-    </link>
--->
     <link name="base_link">
       <xacro:make_cylinder radius="${base_size_x}" length="${base_size_y}" mass="${base_mass}" xyz="${base_x} ${base_y} ${base_z}"/>
@@ -60,5 +50,5 @@
       radius="${wheel_radius}" width="${wheel_width}" mass="${wheel_mass}">
       <origin xyz="${wheel_base_x} ${wheel_base_y} ${wheel_base_z}"/>
-    </xacro:wheel>
+    </xacro:wheel>`
     <xacro:wheel wheel_prefix="right" parent_link="base_link" left_right="1"
       radius="${wheel_radius}" width="${wheel_width}" mass="${wheel_mass}">
@@ -73,9 +63,4 @@
       <origin xyz="${-1*wheel_base_x} ${-wheel_base_y} ${wheel_base_z}"/>
     </xacro:wheel>
-    <!--
-    <xacro:roller name="front" parent="base_link" radius="${roller_radius}" mass="${roller_mass}">
-      <origin xyz="${roller_base_x} ${roller_base_y} ${roller_base_z}"/>
-    </xacro:roller>
-    -->
     <!-- ============ Enter sensors code here =============== -->
     <!-- ============ LIDAR =============== -->
